File: megashield/Mega_Shield-v13.sch (EAGLE design)
At the start: 18 parts

Commit message: Updates to board
Parts:
- removed U$1: LOGO-SFENEW, SparkFun:LOGO-SFENEW
Changed lines of the file:
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@@
 <parts>
 <part name="FRAME1" library="SparkFun" deviceset="FRAME-LETTER" device=""/>
-<part name="U$1" library="SparkFun" deviceset="LOGO-SFE" device="NEW"/>
 <part name="JP3" library="SparkFun" deviceset="M08" device="LOCK"/>
 <part name="JP4" library="SparkFun" deviceset="M08" device="LOCK"/>
@@
 <instance part="FRAME1" gate="G$1" x="0" y="0"/>
 <instance part="FRAME1" gate="G$2" x="147.32" y="0"/>
-<instance part="U$1" gate="G$1" x="152.4" y="27.94"/>
 <instance part="JP3" gate="G$1" x="81.28" y="129.54" rot="R90"/>
 <instance part="JP4" gate="G$1" x="111.76" y="129.54" rot="R90"/>
