File: megashield/Mega_Shield-v13.brd (EAGLE design)
At the start: 101.6 x 53.3 mm, 18 parts

Commit message: Major changes to the layout...
Parts:
- removed U$1: LOGO-SFENEW, SparkFun:SFE-NEW-WEBLOGO
Routing:
- net GND: track 0.00 -> 6.35 mm, vias 11 -> 13
- net N$8: track 0.00 -> 5.08 mm, vias 1 -> 3
- net N$6: track 0.00 -> 5.08 mm, vias 1 -> 3
- net N$410: track 0.00 -> 5.08 mm, vias 1 -> 3
- net N$41: track 0.00 -> 5.08 mm, vias 0 -> 3
- net N$403: track 0.00 -> 5.08 mm, vias 1 -> 3
- net N$400: track 0.00 -> 5.08 mm, vias 1 -> 3
- net N$40: track 0.00 -> 5.08 mm, vias 0 -> 3
- net N$4: track 0.00 -> 5.08 mm, vias 1 -> 3
- net N$21: track 0.00 -> 5.08 mm, vias 1 -> 3
- net N$19: track 0.00 -> 5.08 mm, vias 1 -> 3
- net N$15: track 0.00 -> 5.08 mm, vias 1 -> 3
- net N$14: track 0.00 -> 5.08 mm, vias 1 -> 3
- net N$13: track 0.00 -> 5.08 mm, vias 1 -> 3
- net N$10: track 0.00 -> 5.08 mm, vias 1 -> 3
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Other:
- board text added: "3/8/2012"
- board text added: "Analog"
- board text added: "http://chrisd.info/portfolio cjd@chrisd.info"
- board text removed: "31"
- board text removed: "33"
- board text removed: "35"
- board text removed: "37"
- board text removed: "39"
- board text removed: "41"
- board text removed: "43"
- board text removed: "45"
- board text removed: "47"
- board text removed: "49"
- board text removed: "51"
- board text removed: "53"
- board text removed: "7/8/09"
- board text removed: "ANALOG IN"
- board text removed: "Arduino Mega ProtoShield"
- board text removed: "COMMUNICATION"
- board text removed: "DIGITAL"
- board text removed: "PWM"
- board text removed: "RX"
- board text removed: "RX1"
- board text removed: "RX2"
- board text removed: "RX3"
- board text removed: "SCL"
- board text removed: "SDA"
- board text removed: "TX"
- board text removed: "TX1"
- board text removed: "TX2"
- board text removed: "TX3"

Commit message: Minor updates to the layout, added an image
Routing:
- net N$72: track 0.00 -> 2.54 mm, vias 1 -> 2
- net N$71: track 0.00 -> 2.54 mm, vias 1 -> 2
- net N$44: track 0.00 -> 2.54 mm, vias 1 -> 2
- net N$111: track 0.00 -> 2.54 mm, vias 1 -> 2
- net N$110: track 0.00 -> 2.54 mm, vias 1 -> 2
- net N$109: track 0.00 -> 2.54 mm, vias 1 -> 2
- net N$108: track 0.00 -> 2.54 mm, vias 1 -> 2
- net N$107: track 0.00 -> 2.54 mm, vias 1 -> 2
- net N$165: track 0.00 -> 2.54 mm, vias 1 -> 2
- net N$162: track 0.00 -> 2.54 mm, vias 1 -> 2
- net N$141: track 0.00 -> 2.54 mm, vias 0 -> 2
- net N$137: track 0.00 -> 2.54 mm, vias 1 -> 2
- net N$136: track 0.00 -> 2.54 mm, vias 1 -> 2
- net N$116: track 0.00 -> 2.54 mm, vias 1 -> 2
- net N$115: track 0.00 -> 2.54 mm, vias 1 -> 2
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Other:
- board text added: "3.3V Bus"
- board text removed: "3.3"
